File: schem/schem.kicad_sch (KiCad schematic)
At the start: 1 part, among them U1 N76E003AT20

Commit message: Add files via upload
Parts:
- added SW1: START_BUTTON, symbol Switch:SW_Push
- added SW2: MODE_BUTTON, symbol Switch:SW_Push
- added SW3: TENS_BUTTON, symbol Switch:SW_Push
- added SW4: ONES_BUTTON, symbol Switch:SW_Push
- added U2: OP07, symbol Amplifier_Operational:OP07
- added U3: LMC7660, symbol Regulator_SwitchedCapacitor:LMC7660
Connections:
- net GND: now also U2.4 (V-); no longer U1.20 (P0.4/AIN5/STADC/PWM3/IC3)
- net at U1.11 (P1.4/SDA/FB/PWM1): now also U1.16 (P0.0/PWM3/IC3/MOSI/T1), U1.17 (P0.1/PWM4/IC4/MISO), U1.18 (P0.2/ICPCK/OCDCK/RXD_1/[SCL]), U1.19 (P0.3/PWM5/IC5/AIN6)
- new net: SW1.1, SW1.2
- new net Alumel: U2.2 (-)
- new net Chromel: U2.3 (+)
- no-connect marks 0 -> 5
Other:
- note removed: "LCD_D4"
- note removed: "LCD_D5"
- note removed: "LCD_D6"
- note removed: "LCD_D7"
- note removed: "LCD_E"
- note removed: "LCD_RS"
- note removed: "RST"
- note removed: "RXD"
- note removed: "TXD"
- moved on the sheet: U1

Commit message: Add files via upload
Parts:
- added J1: LCM-S01602DTR_M, LCM-S01602DTR_M:LCD_LCM-S01602DTR_M, symbol LCM-S01602DTR_M:LCM-S01602DTR_M
- added R1: 10kΩ, symbol Device:R
- added SW1: Reset, symbol Switch:SW_Push
- added SW5: Boot, symbol Switch:SW_Push
Connections:
- net GND is gone; now on net Earth: U2.4 (V-)
- net +5V: now also U2.7 (V+)
- net at U1.12 (P1.3/SCL/[STADC): now also J1.6 (E)
- net RXD: now reaches U1.2 (TXD/AIN3/P0.6)
- net RXD: now also R1.1
- net TXD: now reaches U1.3 (RXD/AIN2/P0.7)
- net CBUS3: now reaches U1.4 (RST/P2.0)
- net CBUS3: now also SW1.1
- net Earth: now reaches U1.7 (GND)
- net Earth: now also SW1.2, SW5.2
- new net: J1.11 (DB4), U1.16 (P0.0/PWM3/IC3/MOSI/T1)
- new net: J1.12 (DB5), U1.17 (P0.1/PWM4/IC4/MISO)
- new net: J1.13 (DB6), U1.18 (P0.2/ICPCK/OCDCK/RXD_1/[SCL])
- new net: J1.14 (DB7), U1.19 (P0.3/PWM5/IC5/AIN6)
- new net: J1.4 (RS), U1.11 (P1.4/SDA/FB/PWM1)
- new net CBUS0: R1.2, SW5.1
- no-connect marks 5 -> 0
Other:
- note added: "BO230XS"
